Commit message: addapt urdf models

File: robotino_5dof_moveit_config/urdf/robotino.urdf (robot description, URDF)
Before this commit: robot robot, 13 links, 12 joints
Links:
- link base: geometry visual box size=0.04096 0.0473 0.105
- link link1: geometry collision mesh filename=package://robotino_arm_description/meshes/link1_collision.s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; visual mesh filename=package://robotino_arm_description/meshes/link1.stl
- link link2: geometry collision mesh filename=package://robotino_arm_description/meshes/link2_collision.s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; visual mesh filename=package://robotino_arm_description/meshes/link2.stl
- link link3: geometry collision mesh filename=package://robotino_arm_description/meshes/link3_collision.s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; visual mesh filename=package://robotino_arm_description/meshes/link3.stl
- link link4: geometry collision mesh filename=package://robotino_arm_description/meshes/link4_collision.s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; visual mesh filename=package://robotino_arm_description/meshes/link4.stl
- link motor1: geometry collision mesh filename=package://robotino_arm_description/meshes/motor1_collision.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; visual mesh filename=package://robotino_arm_description/meshes/motor1.stl
- link motor2: geometry visual box size=0 0 0
Joints:
- joint joint2: limit lower=-2.443460952792061 upper=2.443460952792061 effort=190 velocity=30 -> lower=-1.9 upper=1.9 effort=190 velocity=30
- joint joint3: limit lower=-3.141592653589793 upper=3.141592653589793 effort=190 velocity=30 -> lower=-1.7 upper=1.7 effort=190 velocity=30
- joint joint4: limit lower=-3.141592653589793 upper=3.141592653589793 effort=160 velocity=30 -> lower=-1.7 upper=1.7 effort=160 velocity=30
- joint joint5: limit lower=-3.141592653589793 upper=3.141592653589793 effort=160 velocity=30 -> lower=-1.7 upper=1.7 effort=160 velocity=30

File: robotino_6dof_moveit_config/urdf/robotino.urdf (robot description, URDF)
Before this commit: robot robot, 14 links, 13 joints
Links:
- link base: geometry visual box size=0.04096 0.0473 0.105
- link link1: geometry collision mesh filename=package://robotino_arm_description/meshes/link1_collision.s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; visual mesh filename=package://robotino_arm_description/meshes/link1.stl
- link link2: geometry collision mesh filename=package://robotino_arm_description/meshes/link2_collision.s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; visual mesh filename=package://robotino_arm_description/meshes/link2.stl
- link link3: geometry collision mesh filename=package://robotino_arm_description/meshes/link3_collision.s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; visual mesh filename=package://robotino_arm_description/meshes/link3.stl
- link link4: geometry collision mesh filename=package://robotino_arm_description/meshes/link4_collision.s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; visual mesh filename=package://robotino_arm_description/meshes/link4.stl
- link motor1: geometry collision mesh filename=package://robotino_arm_description/meshes/motor1_collision.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; visual mesh filename=package://robotino_arm_description/meshes/motor1.stl
- link motor2: geometry visual box size=0 0 0
Joints:
- joint joint2: limit lower=-2.443460952792061 upper=2.443460952792061 effort=190 velocity=30 -> lower=-1.9 upper=1.9 effort=190 velocity=30
- joint joint3: limit lower=-3.141592653589793 upper=3.141592653589793 effort=190 velocity=30 -> lower=-1.7 upper=1.7 effort=190 velocity=30
- joint joint4: limit lower=-3.141592653589793 upper=3.141592653589793 effort=160 velocity=30 -> lower=-1.7 upper=1.7 effort=160 velocity=30
- joint joint5: limit lower=-3.141592653589793 upper=3.141592653589793 effort=160 velocity=30 -> lower=-1.7 upper=1.7 effort=160 velocity=30

File: uibk_robotino2_5dof_moveit_config/urdf/robotino.urdf (robot description, URDF)
Before this commit: robot robot, 30 links, 29 joints
Links:
- link base: geometry visual box size=0.04096 0.0473 0.105
- link hand_left_coupler: geometry collision mesh filename=package://kclhand_description/meshes/left_coupler.STL; visual mesh filename=package://kclhand_description/meshes/left_coupler.STL
- link hand_left_crank: geometry collision mesh filename=package://kclhand_description/meshes/left_crank.STL; visual mesh filename=package://kclhand_description/meshes/left_crank.STL
- link hand_left_finger_lower_link: geometry collision mesh filename=package://kclhand_description/meshes/left_finger_lower_link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; visual mesh filename=package://kclhand_description/meshes/left_finger_lower_link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
- link hand_left_finger_upper_link: geometry collision mesh filename=package://kclhand_description/meshes/left_finger_upper_link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; visual mesh filename=package://kclhand_description/meshes/left_finger_upper_link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
- link hand_middle_finger_lower_link: geometry collision mesh filename=package://kclhand_description/meshes/middle_finger_lower_li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; visual mesh filename=package://kclhand_description/meshes/middle_finger_lower_li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
- link hand_middle_finger_upper_link: geometry collision mesh filename=package://kclhand_description/meshes/middle_finger_upper_li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; visual mesh filename=package://kclhand_description/meshes/middle_finger_upper_li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
- link hand_right_coupler: geometry collision mesh filename=package://kclhand_description/meshes/right_coupler.STL; visual mesh filename=package://kclhand_description/meshes/right_coupler.STL
- link hand_right_crank: geometry collision mesh filename=package://kclhand_description/meshes/right_crank.STL; visual mesh filename=package://kclhand_description/meshes/right_crank.STL
- link hand_right_finger_lower_link: geometry collision mesh filename=package://kclhand_description/meshes/right_finger_lower_lin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; visual mesh filename=package://kclhand_description/meshes/right_finger_lower_lin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
- link hand_right_finger_upper_link: geometry collision mesh filename=package://kclhand_description/meshes/right_finger_upper_lin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; visual mesh filename=package://kclhand_description/meshes/right_finger_upper_lin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
- link link1: geometry collision mesh filename=package://robotino_arm_description/meshes/link1_collision.s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; visual mesh filename=package://robotino_arm_description/meshes/link1.stl
- link link2: geometry collision mesh filename=package://robotino_arm_description/meshes/link2_collision.s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; visual mesh filename=package://robotino_arm_description/meshes/link2.stl
- link link3: geometry collision mesh filename=package://robotino_arm_description/meshes/link3_collision.s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; visual mesh filename=package://robotino_arm_description/meshes/link3.stl
- link link4: geometry collision mesh filename=package://robotino_arm_description/meshes/link4_collision.s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; visual mesh filename=package://robotino_arm_description/meshes/link4.stl
- link motor1: geometry collision mesh filename=package://robotino_arm_description/meshes/motor1_collision.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; visual mesh filename=package://robotino_arm_description/meshes/motor1.stl
- link motor2: geometry visual box size=0 0 0
Joints:
- joint base_pan_joint: origin xyz=0.203 0.003 0.55 rpy=0 0 0.0 -> xyz=0 0 0 rpy=0 0 0
- joint hokuyo_joint: origin xyz=0.064 0.0 0.22 rpy=0.0 0.0 0.0 -> xyz=0.11 0.05 0.105 rpy=0.0 0.0 -0.0004
- joint joint2: limit lower=-2.443460952792061 upper=2.443460952792061 effort=190 velocity=30 -> lower=-1.9 upper=1.9 effort=190 velocity=30
- joint joint3: limit lower=-3.141592653589793 upper=3.141592653589793 effort=190 velocity=30 -> lower=-1.7 upper=1.7 effort=190 velocity=30
- joint joint4: limit lower=-3.141592653589793 upper=3.141592653589793 effort=160 velocity=30 -> lower=-1.7 upper=1.7 effort=160 velocity=30
- joint joint5: limit lower=-3.141592653589793 upper=3.141592653589793 effort=160 velocity=30 -> lower=-1.7 upper=1.7 effort=160 velocity=30
- joint kinect_joint: origin xyz=0.0 0.065 0.0 rpy=-1.570795 0 0.0 -> xyz=0.0521788 0.174338 -0.064193 rpy=1.57128 -3.08083 3.01699
- joint pan_joint: origin xyz=0 0 0 rpy=0 0 0 -> xyz=0.142355 0.0508101 0.583959 rpy=0.0870705 0.263353 0.33492
