Commit message: updates moveit config

File: robotino_6dof_moveit_config/urdf/robotino.urdf (robot description, URDF)
Before this commit: robot robot, 14 links, 13 joints
Links:
- added link base_pan_link, mass 0.00001; collision box size=0.001 0.001 0.001; visual box size=0.001 0.001 0.001
- added link hand_base_link, mass 0.090062; collision mesh filename=package://kclhand_description/meshes/base_link.STL; visual mesh filename=package://kclhand_description/meshes/base_link.STL
- added link hand_cableCanal_link, mass 0.090062; collision mesh filename=package://kclhand_description/meshes/cableCanalCollision.stl; visual box size=0.0 0.0 0.0
- added link hand_left_coupler, mass 0.01251; collision mesh filename=package://kclhand_description/meshes/left_coupler.STL; visual mesh filename=package://kclhand_description/meshes/left_coupler.STL
- added link hand_left_crank, mass 0.0043398; collision mesh filename=package://kclhand_description/meshes/left_crank.STL; visual mesh filename=package://kclhand_description/meshes/left_crank.STL
- added link hand_left_finger_lower_link, mass 0.006486; collision mesh filename=package://kclhand_description/meshes/left_finger_lower_link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; visual mesh filename=package://kclhand_description/meshes/left_finger_lower_link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
- added link hand_left_finger_upper_link, mass 0.0074578; collision mesh filename=package://kclhand_description/meshes/left_finger_upper_link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; visual mesh filename=package://kclhand_description/meshes/left_finger_upper_link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
- added link hand_middle_finger_lower_link, mass 0.006486; collision mesh filename=package://kclhand_description/meshes/middle_finger_lower_li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; visual mesh filename=package://kclhand_description/meshes/middle_finger_lower_li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
- added link hand_middle_finger_upper_link, mass 0.0074578; collision mesh filename=package://kclhand_description/meshes/middle_finger_upper_li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; visual mesh filename=package://kclhand_description/meshes/middle_finger_upper_li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
- added link hand_right_coupler, mass 0.011998; collision mesh filename=package://kclhand_description/meshes/right_coupler.STL; visual mesh filename=package://kclhand_description/meshes/right_coupler.STL
- added link hand_right_crank, mass 0.0043398; collision mesh filename=package://kclhand_description/meshes/right_crank.STL; visual mesh filename=package://kclhand_description/meshes/right_crank.STL
- added link hand_right_finger_lower_link, mass 0.006486; collision mesh filename=package://kclhand_description/meshes/right_finger_lower_lin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; visual mesh filename=package://kclhand_description/meshes/right_finger_lower_lin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
- added link hand_right_finger_upper_link, mass 0.00745775236371133; collision mesh filename=package://kclhand_description/meshes/right_finger_upper_lin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; visual mesh filename=package://kclhand_description/meshes/right_finger_upper_lin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
- added link hand_wrist_link, mass 0.090062; collision mesh filename=package://kclhand_description/meshes/wrist.stl; visual mesh filename=package://kclhand_description/meshes/wrist.stl
- added link kinect_link, mass 0.00001; collision box size=0.035 0.18 0.02; visual box size=0.035 0.18 0.02
- added link pan_link, mass 0.00001
- added link profile_link, mass 0.00001; collision mesh filename=package://robotino_description/meshes/pan_tilt_tuw.stl; visual mesh filename=package://robotino_description/meshes/pan_tilt_tuw.stl
- added link tilt_link, mass 0.00001
Joints:
- added joint base_pan_joint: type fixed, parent profile_link, child base_pan_link, origin xyz=0.145 0.194 0.64 rpy=0.0 0.0 1.0472
- added joint hand_base_joint: type fixed, parent hand_wrist_link, child hand_base_link, origin xyz=-0.02105 0.1485 0 rpy=0 0.52 0
- added joint hand_cableCanal_joint: type fixed, parent hand_wrist_link, child hand_cableCanal_link, origin xyz=0 0.06 0.07 rpy=0 0 0
- added joint hand_left_coupler_crank_joint: type continuous, parent hand_left_crank, child hand_left_coupler, origin xyz=0 0 0 rpy=0.40154 0.63113 0.62376, axis 0 0 1
- added joint hand_left_crank_base_joint: type continuous, parent hand_base_link, child hand_left_crank, origin xyz=0 0 0 rpy=-2.1588 0.44783 -1.8518, axis 0 0 1
- added joint hand_left_finger_lower_joint: type continuous, parent hand_left_coupler, child hand_left_finger_lower_link, origin xyz=0.016246 0.021 0.044635 rpy=-1.2217 -7.6328E-17 1.5708, axis 0 0 -1
- added joint hand_left_finger_upper_joint: type continuous, parent hand_left_finger_lower_link, child hand_left_finger_upper_link, origin xyz=0.05 0 0 rpy=-1.5543E-15 7.7716E-16 0.7854, axis 0 0 1
- added joint hand_middle_finger_lower_joint: type continuous, parent hand_base_link, child hand_middle_finger_lower_link, origin xyz=0.035507 0.02 0.0205 rpy=-0.5236 5.5511E-17 1.5708, axis 0 0 -1
- added joint hand_middle_finger_upper_joint: type continuous, parent hand_middle_finger_lower_link, child hand_middle_finger_upper_link, origin xyz=0.05 0 0 rpy=0 0 0.7854, axis 0 0 1
- added joint hand_right_coupler_crank_joint: type continuous, parent hand_right_crank, child hand_right_coupler, origin xyz=0 0 0 rpy=0.40154 -0.63113 -0.62376, axis 0 0 1
- added joint hand_right_crank_base_joint: type continuous, parent hand_base_link, child hand_right_crank, origin xyz=0 0 0 rpy=-5.5511E-17 -2.7756E-17 1.0472, axis 0 0 1
- added joint hand_right_finger_lower_joint: type continuous, parent hand_right_coupler, child hand_right_finger_lower_link, origin xyz=-0.016246 0.021 0.044635 rpy=-1.9199 -2.047E-16 1.5708, axis 0 0 1
- added joint hand_right_finger_upper_joint: type continuous, parent hand_right_finger_lower_link, child hand_right_finger_upper_link, origin xyz=0.05 0 0 rpy=4.4409E-16 -2.9143E-16 0.7854, axis 0 0 1
- added joint hand_wrist_joint: type fixed, parent link5, child hand_wrist_link, origin xyz=0 0 0 rpy=1.5707963 0 0
- added joint kinect_joint: type fixed, parent tilt_link, child kinect_link, origin xyz=0.03129 0.058 -0.0 rpy=-1.56905 0.0434565 0.00667917
- added joint pan_joint: type revolute, parent base_pan_link, child pan_link, origin xyz=0 0 0 rpy=0 0 0, axis 0 0 1, limit lower=-1.57 upper=1.57 effort=100 velocity=1.4
- added joint profile_joint: type fixed, parent base_link, child profile_link, origin xyz=0 0 0 rpy=0 0 0
- added joint tilt_joint: type revolute, parent pan_link, child tilt_link, origin xyz=0 0 0 rpy=1.57 0 0, axis 0 0 -1, limit lower=-1.57 upper=1.57 effort=100 velocity=1.4
- joint hokuyo_joint: origin xyz=0.064 0.0 0.22 rpy=0.0 0.0 0.0 -> xyz=0.184 0.004 0.16 rpy=0.0 0.0 -0.015

File: uibk_robotino2_moveit_config/urdf/robotino.urdf (robot description, URDF)
Before this commit: robot robot, 30 links, 29 joints
Links:
- added link hand_cableCanal_link, mass 0.090062; collision mesh filename=package://kclhand_description/meshes/cableCanalCollision.stl; visual box size=0.0 0.0 0.0
- added link profile_link, mass 0.00001; collision mesh filename=package://robotino_description/meshes/pan_tilt.stl; visual mesh filename=package://robotino_description/meshes/pan_tilt.stl
- link base_pan_link: geometry collision box size=0.001 0.001 0.001; visual box size=0.001 0.001 0.001
Joints:
- added joint hand_cableCanal_joint: type fixed, parent hand_wrist_link, child hand_cableCanal_link, origin xyz=0 0.06 0.07 rpy=0 0 0
- added joint profile_joint: type fixed, parent base_link, child profile_link, origin xyz=0 0 0 rpy=0 0 0
- joint base_pan_joint: origin xyz=0 0 0 rpy=0 0 0 -> xyz=0.142355 0.0508101 0.583959 rpy=0.0870705 0.263353 0.33492; parent base_link -> profile_link
- joint pan_joint: origin xyz=0.142355 0.0508101 0.583959 rpy=0.0870705 0.263353 0.33492 -> xyz=0 0 0 rpy=0 0 0

Commit message: added a collision case

File: robotino_6dof_moveit_config/urdf/robotino.urdf (robot description, URDF)
Before this commit: robot robot, 32 links, 31 joints
Links:
- added link case_link, mass 4; collision mesh filename=package://robotino_description/meshes/case.stl
Joints:
- added joint case_joint: type fixed, parent base_link, child case_link, origin xyz=0 0 0 rpy=0 0 0

File: uibk_robotino2_moveit_config/urdf/robotino.urdf (robot description, URDF)
Before this commit: robot robot, 32 links, 31 joints
Links:
- added link case_link, mass 4; collision mesh filename=package://robotino_description/meshes/case.stl
Joints:
- added joint case_joint: type fixed, parent base_link, child case_link, origin xyz=0 0 0 rpy=0 0 0
